File: SDSQ1/SDSQ1.kicad_pcb (KiCad board)
At the start: 2 copper layers, 101.5 x 109.1 mm, 129 parts, among them J1 AudioJack2, J3 Jack-DC, Q1 NPN, Q10 NPN, Q11 NPN, Q2 NPN, Q3 NPN, Q4 NPN, Q5 NPN, Q6 NPN, Q7 NPN, Q8 NPN, Q9 NPN, SW1 SW_SPDT, SW10 SW_SPST, SW11 SW_SPST, SW13 SW_SPST, SW14 SW_SPST, SW15 SW_SPST, SW16 SW_SPST, SW18 SW_SPST, SW19 SW_SPST, SW2 SW_SPST, SW20 SW_SPST, SW21 SW_SPST, SW23 SW_SPST, SW24 SW_SPST, SW25 SW_SPST, SW26 SW_SPST, SW28 SW_SPST, SW29 SW_SPST, SW3 SW_SPST, SW30 SW_SPST, SW31 SW_SPST, SW33 SW_SPST, SW34 SW_SPST, SW35 SW_SPST, SW36 SW_SPST, SW38 SW_SPST, SW39 SW_SPST, SW4 SW_SPST, SW40 SW_SPST, SW41 SW_SPST, SW5 SW_SPST, SW6 SW_SPST, SW8 SW_SPST, SW9 SW_SPST, U1 Opamp_Dual, U2 Opamp_Dual, U3 Opamp_Dual, U4 LTC4054ES5-4.2, U5 NCP1117-5.0_SOT223, U6 4017, U7 ICM7555xP

Commit message: removed ignores
Parts:
- added G***: LOGO, LOGO, B.Cu at (94.5, 94.5)
- added REF**: Polarity_Center_Negative_6mm_SilkScreen, Symbol:Polarity_Center_Negative_6mm_SilkScreen, F.Cu at (88.9, 49.3)
- added REF**: OSHW-Logo_38.1x40mm_SilkScreen, Symbol:OSHW-Logo_38.1x40mm_SilkScreen, B.Cu at (141.7, 93.0)
- added REF**: WEEE-Logo_5.6x8mm_SilkScreen, Symbol:WEEE-Logo_5.6x8mm_SilkScreen, B.Cu at (152.4, 47.8)
- added REF**: KiCad-Logo2_5mm_SilkScreen, Symbol:KiCad-Logo2_5mm_SilkScreen, B.Cu at (160.0, 35.1)
Other:
- board text added: "Designed by Nathan Shelburn github.com/Superliminal-Defenestration SD-SQ1-A"
- board text added: "What are you doing here?"
